Commit message: upadted models to humble

File: urdf/test.urdf.xacro (robot description, xacro)
@@ -1,27 +1,26 @@
 <?xml version="1.0"?>
 <robot name="sensor_stack" xmlns:xacro="http://ros.org/wiki/xacro">
-  <xacro:arg name="base_link_name" default="bask_link"/>
+  <!-- Args -->
+  <xacro:arg name="base_link_name" default="base_link"/>
   <xacro:arg name="rot_link" default="rot_link"/>
   <!-- Ouster pose -->
   <xacro:arg name="os1_xyz" default="0.00 0.00 0.09"/>
   <xacro:arg name="os1_rpy" default="0 0 0"/>
-  <!-- ZED2i pose -->
+  <!-- ZED2i pose (mount transform of zed2i_camera_link to rot_link) -->
   <xacro:arg name="zed_xyz" default="0.05 0.00 0.0"/>
   <xacro:arg name="zed_rpy" default="0 0 0"/>
+  <!-- Base links -->
   <link name="$(arg base_link_name)"/>
-    <link name="$(arg rot_link)"/>
+  <link name="$(arg rot_link)"/>
+  <!-- rot_link -> base_link with -15 deg pitch -->
   <joint name="$(arg base_link_name)_joint" type="fixed">
-    <origin xyz="0 0 0" rpy="0 -0.26179 0"/>
-    <parent link="$(arg rot_link)"/>
-    <child link="$(arg base_link_name)"/>
-    </joint>
-  <!--  Include your sensor Xacros (no copy/paste)  -->
+    <origin xyz="0 0 0" rpy="0 0.26179 0"/>
+    <parent link="$(arg base_link_name)"/>
+    <child link="$(arg rot_link)"/>
+  </joint>
+  <!-- Includes -->
   <xacro:include filename="$(find urdf_viewer)/urdf/ouster_os1.urdf.xacro"/>
   <xacro:include filename="$(find urdf_viewer)/urdf/zed_macro.urdf.xacro"/>
-  <!-- NOTE: zed_descr.urdf.xacro is a full robot, not a macro.
-       Don't include it here or you'll get nested <robot> tags.
-       Use the zed_camera macro from zed_macro.urdf.xacro instead. -->
-  <!--  Instantiate sensors on the base  -->
-  <!-- Ouster OS1-64 (macro name matches your file) -->
+  <!-- Ouster OS1-64 -->
   <xacro:OS1-64 parent="$(arg rot_link)"
                 name="os1"
@@ -32,7 +31,17 @@
     <origin xyz="$(arg os1_xyz)" rpy="$(arg os1_rpy)"/>
   </xacro:OS1-64>
-  <!-- ZED2i -->
-  <xacro:zed_camera name="zed2i" model="zed2i" parent="$(arg rot_link)">
+  <!-- ZED2i: instantiate macro (creates zed2i_camera_link …), then mount it -->
+  <xacro:zed_camera name="zed2i" model="zed2i" enable_gnss="false">
+  <!-- block required by *gnss_origin; used only if GNSS is enabled -->
+  <origin xyz="0 0 0" rpy="0 0 0"/>
+</xacro:zed_camera>
+  <!-- Mount ZED to rot_link (this replaces the old 'parent' + nested origin) -->
+  <joint name="zed2i_mount" type="fixed">
+    <parent link="$(arg rot_link)"/>
+    <child  link="zed2i_camera_link"/>
     <origin xyz="$(arg zed_xyz)" rpy="$(arg zed_rpy)"/>
-  </xacro:zed_camera>
+  </joint>
+  <!-- NOTE:
+       Do NOT include zed_descr.urdf.xacro here (it’s a full <robot/> wrapper).
+       Use only zed_macro.urdf.xacro as above. -->
 </robot>

File: urdf/zed_descr.urdf.xacro (robot description, xacro)
@@ -1,5 +1,5 @@
 <?xml version="1.0"?>
 <!--
-// Copyright 2022 Stereolabs
+// Copyright 2024 Stereolabs
 //
 // Licensed under the Apache License, Version 2.0 (the "License");
@@ -18,19 +18,13 @@
   <xacro:arg name="camera_name"   default="zed" />
   <xacro:arg name="camera_model"  default="zed" />
-  <xacro:arg name="base_frame"    default="base_link" />
-  <xacro:arg name="cam_pos_x"     default="0.0" />
-  <xacro:arg name="cam_pos_y"     default="0.0" />
-  <xacro:arg name="cam_pos_z"     default="0.0" />
-  <xacro:arg name="cam_roll"      default="0.0" />
-  <xacro:arg name="cam_pitch"     default="0.0" />
-  <xacro:arg name="cam_yaw"       default="0.0" />
-  <xacro:arg name="gnss_frame"    default="" />
-  <xacro:include filename="$(find urdf_viewer)/urdf/zed_macro.urdf.xacro" />
-  <xacro:zed_camera name="$(arg camera_name)" model="$(arg camera_model)" parent="$(arg base_frame)">
-    <origin
-      xyz="$(arg cam_pos_x) $(arg cam_pos_y) $(arg cam_pos_z)"
-      rpy="$(arg cam_roll) $(arg cam_pitch) $(arg cam_yaw)"
-    />
+  <xacro:arg name="custom_baseline"  default="0.0" />
+  <!-- If GNSS fusion is enabled the position of the antenna with respect to the camera mount point is required -->
+  <xacro:arg name="enable_gnss"   default="false" />
+  <xacro:arg name="gnss_x" default="0.0" />
+  <xacro:arg name="gnss_y" default="0.0" />
+  <xacro:arg name="gnss_z" default="0.0" />
+  <xacro:include filename="$(find zed_wrapper)/urdf/zed_macro.urdf.xacro" />
+  <xacro:zed_camera name="$(arg camera_name)" model="$(arg camera_model)" custom_baseline="$(arg custom_baseline)" enable_gnss="$(arg enable_gnss)">
+	    <origin xyz="$(arg gnss_x) $(arg gnss_y) $(arg gnss_z)" rpy="0 0 0"/>
   </xacro:zed_camera>
-  <link name="$(arg base_frame)" />
 </robot>

File: urdf/zed_macro.urdf.xacro (robot description, xacro)
@@ -1,5 +1,5 @@
 <?xml version="1.0"?>
 <!--
-// Copyright 2022 Stereolabs
+// Copyright 2024 Stereolabs
 //
 // Licensed under the Apache License, Version 2.0 (the "License");
@@ -21,9 +21,8 @@
     Parameters:
       - name: the camera's name.  should match the parameter sent to the launch file for this camera
-      - model: the tye of camera, one of zed, zedm, zed2, zed2i
-      - parent: the parent link of the camera.  must be defined in the URDF file that uses this macro
-      - origin: the xyz/rpy offset from the parent link
+      - model: the type of camera, one of zed, zedm, zed2, zed2i, zedx, zedxm, virtual
+      - enable_gnss: if true enable the URDF link
   -->
-  <xacro:macro name="zed_camera" params="name=zed model=zed parent *origin">
+  <xacro:macro name="zed_camera" params="name=zed model=zed enable_gnss=false custom_baseline=0 *gnss_origin">
     <xacro:if value="${model == 'zed'}">
       <xacro:property name="baseline" value="0.12" />
@@ -33,7 +32,8 @@
       <xacro:property name="screw_offset_z" value="0.0" />
       <xacro:property name="optical_offset_x" value="-0.01" />
+      <xacro:property name="mono" value="false" />
     </xacro:if>
     <xacro:if value="${model == 'zedm'}">
-      <xacro:property name="baseline" value="0.06" />
+      <xacro:property name="baseline" value="0.063" />
       <xacro:property name="height" value="0.0265" />
       <xacro:property name="bottom_slope" value="0.0" />
@@ -41,4 +41,5 @@
       <xacro:property name="screw_offset_z" value="0.0" />
       <xacro:property name="optical_offset_x" value="0.0" />
+      <xacro:property name="mono" value="false" />
     </xacro:if>
     <xacro:if value="${model == 'zed2'}">
@@ -49,4 +50,5 @@
       <xacro:property name="screw_offset_z" value="0.0" />
       <xacro:property name="optical_offset_x" value="-0.01" />
+      <xacro:property name="mono" value="false" />
     </xacro:if>
     <xacro:if value="${model == 'zed2i'}">
@@ -57,4 +59,5 @@
       <xacro:property name="screw_offset_z" value="0.0" />
       <xacro:property name="optical_offset_x" value="-0.01" />
+      <xacro:property name="mono" value="false" />
     </xacro:if>
     <xacro:if value="${model == 'zedx'}">
@@ -65,4 +68,5 @@
       <xacro:property name="screw_offset_z" value="-0.016" />
       <xacro:property name="optical_offset_x" value="-0.01" />
+      <xacro:property name="mono" value="false" />
     </xacro:if>
     <xacro:if value="${model == 'zedxm'}">
@@ -73,83 +77,166 @@
       <xacro:property name="screw_offset_z" value="-0.016" />
       <xacro:property name="optical_offset_x" value="-0.01" />
+      <xacro:property name="mono" value="false" />
+    </xacro:if>
+    <xacro:if value="${model == 'virtual'}">
+      <xacro:property name="baseline" value="${custom_baseline}" />
+      <xacro:property name="height" value="0.031" />
+      <xacro:property name="bottom_slope" value="0.0" />
+      <xacro:property name="screw_offset_x" value="0.00" />
+      <xacro:property name="screw_offset_z" value="-0.0155" />
+      <xacro:property name="optical_offset_x" value="0.0" />
+      <xacro:property name="mono" value="false" />
+    </xacro:if>
+    <xacro:if value="${model == 'zedxonegs'}">
+      <xacro:property name="baseline" value="0.0" />
+      <xacro:property name="height" value="0.031" />
+      <xacro:property name="bottom_slope" value="0.0" />
+      <xacro:property name="screw_offset_x" value="0.0" />
+      <xacro:property name="screw_offset_z" value="-0.0155" />
+      <xacro:property name="optical_offset_x" value="0.0" />
+      <xacro:property name="mono" value="true" />
+    </xacro:if>
+    <xacro:if value="${model == 'zedxone4k'}">
+      <xacro:property name="baseline" value="0.0" />
+      <xacro:property name="height" value="0.031" />
+      <xacro:property name="bottom_slope" value="0.0" />
+      <xacro:property name="screw_offset_x" value="0.00" />
+      <xacro:property name="screw_offset_z" value="-0.0155" />
+      <xacro:property name="optical_offset_x" value="0.0" />
+      <xacro:property name="mono" value="true" />
     </xacro:if>
     <!-- Camera mounting point (the threaded screw hole in the bottom) -->
-    <link name="${name}_base_link" />
-    <joint name="${name}_base_joint" type="fixed">
-      <parent link="${parent}"/>
-      <child link="${name}_base_link"/>
-      <xacro:insert_block name="origin" />
-    </joint>
+    <link name="${name}_camera_link" />
     <!-- Camera Center -->
     <link name="${name}_camera_center">
-      <visual>
-        <origin xyz="${screw_offset_x} 0 ${screw_offset_z}" rpy="0 0 0"/>
-        <geometry>
-          <mesh filename="package://urdf_viewer/meshes/${model}.stl" />
-        </geometry>
-        <material name="${model}_mat" />
-      </visual>
-      <collision>
-        <geometry>
-          <mesh filename="package://urdf_viewer/meshes/${model}.stl" />
-        </geometry>
-      </collision>
+      <xacro:unless value="${model == 'virtual'}">
+        <visual>
+          <origin xyz="${screw_offset_x} 0 ${screw_offset_z}" rpy="0 0 0"/>
+          <geometry>
+<mesh filename="file://$(find urdf_viewer)/meshes/${model}.stl"/>
+          </geometry>
+          <material name="${model}_mat" />
+        </visual>
+        <collision>
+          <origin xyz="${screw_offset_x} 0 ${screw_offset_z}" rpy="0 0 0"/>
+          <geometry>
+<mesh filename="file://$(find urdf_viewer)/meshes/${model}.stl"/>
+          </geometry>
+        </collision>
+      </xacro:unless>
     </link>
     <joint name="${name}_camera_center_joint" type="fixed">
-      <parent link="${name}_base_link"/>
+      <parent link="${name}_camera_link"/>
       <child link="${name}_camera_center"/>
       <origin xyz="0 0 ${height/2}" rpy="0 ${bottom_slope} 0" />
     </joint>
-    <!-- Left Camera -->
-    <link name="${name}_left_camera_frame" />
-    <joint name="${name}_left_camera_joint" type="fixed">
-      <parent link="${name}_camera_center"/>
-      <child link="${name}_left_camera_frame"/>
-      <origin xyz="${optical_offset_x} ${baseline/2} 0" rpy="0 0 0" />
-    </joint>
-    <link name="${name}_left_camera_optical_frame"/>
-    <joint name="${name}_left_camera_optical_joint" type="fixed">
-      <origin xyz="0 0 0" rpy="-${M_PI/2} 0.0 -${M_PI/2}"/>
-      <parent link="${name}_left_camera_frame"/>
-      <child link="${name}_left_camera_optical_frame"/>
-    </joint>
-    <!-- Right Camera -->
-    <link name="${name}_right_camera_frame" />
-    <joint name="${name}_right_camera_joint" type="fixed">
-      <parent link="${name}_camera_center"/>
-      <child link="${name}_right_camera_frame"/>
-      <origin xyz="${optical_offset_x} -${baseline/2} 0" rpy="0 0 0" />
-    </joint>
-    <link name="${name}_right_camera_optical_frame"/>
-    <joint name="${name}_right_camera_optical_joint" type="fixed">
-      <origin xyz="0 0 0" rpy="-${M_PI/2} 0.0 -${M_PI/2}"/>
-      <parent link="${name}_right_camera_frame"/>
-      <child link="${name}_right_camera_optical_frame"/>
-    </joint>
-    <!-- ZED2 Sensors -->
-    <xacro:if value="${model == 'zed2'}">
-      <link name="${name}_mag_link" />
-      <joint name="${name}_mag_joint" type="fixed">
+    <xacro:unless value="${mono}">
+      <!-- Left Camera -->
+      <link name="${name}_left_camera_frame">
+        <xacro:if value="${model == 'virtual'}">
+          <visual>
+            <origin xyz="0 0 0" rpy="0 0 0"/>
+            <geometry>
+  <mesh filename="file://$(find urdf_viewer)/meshes/${model}.stl"/>
+            </geometry>
+            <material name="${model}_mat" />
+          </visual>
+          <collision>
+            <origin xyz="0 0 0" rpy="0 0 0"/>
+            <geometry>
+  <mesh filename="file://$(find urdf_viewer)/meshes/${model}.stl"/>
+            </geometry>
+          </collision>
+        </xacro:if>
+      </link>
+      <joint name="${name}_left_camera_joint" type="fixed">
         <parent link="${name}_camera_center"/>
-        <child link="${name}_mag_link"/>
-        <origin xyz="0 0 0" rpy="0 0 0" />
-      </joint>
-      <link name="${name}_baro_link" />
-      <joint name="${name}_baro_joint" type="fixed">
+        <child link="${name}_left_camera_frame"/>
+        <origin xyz="${optical_offset_x} ${baseline/2} 0" rpy="0 0 0" />
+      </joint>
+      <link name="${name}_left_camera_optical_frame"/>
+      <joint name="${name}_left_camera_optical_joint" type="fixed">
+        <origin xyz="0 0 0" rpy="-${M_PI/2} 0.0 -${M_PI/2}"/>
+        <parent link="${name}_left_camera_frame"/>
+        <child link="${name}_left_camera_optical_frame"/>
+      </joint>
+      <!-- Right Camera -->
+      <link name="${name}_right_camera_frame">
+        <xacro:if value="${model == 'virtual'}">
+          <visual>
+            <origin xyz="0 0 0" rpy="0 0 0"/>
+            <geometry>
+  <mesh filename="file://$(find urdf_viewer)/meshes/${model}.stl"/>
+            </geometry>
+            <material name="${model}_mat" />
+          </visual>
+          <collision>
+            <origin xyz="0 0 0" rpy="0 0 0"/>
+            <geometry>
+  <mesh filename="file://$(find urdf_viewer)/meshes/${model}.stl"/>
+            </geometry>
+          </collision>
+        </xacro:if>
+      </link>
+      <joint name="${name}_right_camera_joint" type="fixed">
         <parent link="${name}_camera_center"/>
-        <child link="${name}_baro_link"/>
-        <origin xyz="0 0 0" rpy="0 0 0" />
-      </joint>
-      <link name="${name}_temp_left_link" />
-      <joint name="${name}_temp_left_joint" type="fixed">
-        <parent link="${name}_left_camera_frame"/>
-        <child link="${name}_temp_left_link"/>
-        <origin xyz="0 0 0" rpy="0 0 0" />
-      </joint>
-      <link name="${name}_temp_right_link" />
-      <joint name="${name}_temp_right_joint" type="fixed">
+        <child link="${name}_right_camera_frame"/>
+        <origin xyz="${optical_offset_x} -${baseline/2} 0" rpy="0 0 0" />
+      </joint>
+      <link name="${name}_right_camera_optical_frame"/>
+      <joint name="${name}_right_camera_optical_joint" type="fixed">
+        <origin xyz="0 0 0" rpy="-${M_PI/2} 0.0 -${M_PI/2}"/>
         <parent link="${name}_right_camera_frame"/>
-        <child link="${name}_temp_right_link"/>
-        <origin xyz="0 0 0" rpy="0 0 0" />
+        <child link="${name}_right_camera_optical_frame"/>
+      </joint>
+      <!-- ZED2 Sensors -->
+      <xacro:if value="${model == 'zed2'}">
+        <link name="${name}_mag_link" />
+        <joint name="${name}_mag_joint" type="fixed">
+          <parent link="${name}_camera_center"/>
+          <child link="${name}_mag_link"/>
+          <origin xyz="0 0 0" rpy="0 0 0" />
+        </joint>
+        <link name="${name}_baro_link" />
+        <joint name="${name}_baro_joint" type="fixed">
+          <parent link="${name}_camera_center"/>
+          <child link="${name}_baro_link"/>
+          <origin xyz="0 0 0" rpy="0 0 0" />
+        </joint>
+        <link name="${name}_temp_left_link" />
+        <joint name="${name}_temp_left_joint" type="fixed">
+          <parent link="${name}_left_camera_frame"/>
+          <child link="${name}_temp_left_link"/>
+          <origin xyz="0 0 0" rpy="0 0 0" />
+        </joint>
+        <link name="${name}_temp_right_link" />
+        <joint name="${name}_temp_right_joint" type="fixed">
+          <parent link="${name}_right_camera_frame"/>
+          <child link="${name}_temp_right_link"/>
+          <origin xyz="0 0 0" rpy="0 0 0" />
+        </joint>
+      </xacro:if>
+    </xacro:unless>
+    <xacro:if value="${mono}">
+      <!-- Camera -->
+      <link name="${name}_camera_frame" />
+      <joint name="${name}_camera_joint" type="fixed">
+        <parent link="${name}_camera_center"/>
+        <child link="${name}_camera_frame"/>
+        <origin xyz="${optical_offset_x} 0 0" rpy="0 0 0" />
+      </joint>
+      <link name="${name}_camera_optical_frame"/>
+      <joint name="${name}_camera_optical_joint" type="fixed">
+        <origin xyz="0 0 0" rpy="-${M_PI/2} 0.0 -${M_PI/2}"/>
+        <parent link="${name}_camera_frame"/>
+        <child link="${name}_camera_optical_frame"/>
+      </joint>
+    </xacro:if>
+    <xacro:if value="${enable_gnss}">
+      <link name="${name}_gnss_link" />
+      <joint name="${name}_gnss_joint" type="fixed">
+        <parent link="${name}_camera_link"/>
+        <child link="${name}_gnss_link"/>
+        <xacro:insert_block name="gnss_origin" />
       </joint>
     </xacro:if>

Commit message: modfied names

File: urdf/test.urdf.xacro (robot description, xacro)
@@ -24,20 +24,20 @@
   <!-- Ouster OS1-64 -->
   <xacro:OS1-64 parent="$(arg rot_link)"
-                name="os1"
+                name="os_sensor"
                 topic_points="/os1/points"
                 topic_imu="/os1/imu"
-                lidar_link="os1_lidar"
-                imu_link="os1_imu">
+                lidar_link="os_lidar"
+                imu_link="os_imu">
     <origin xyz="$(arg os1_xyz)" rpy="$(arg os1_rpy)"/>
   </xacro:OS1-64>
   <!-- ZED2i: instantiate macro (creates zed2i_camera_link …), then mount it -->
-  <xacro:zed_camera name="zed2i" model="zed2i" enable_gnss="false">
+  <xacro:zed_camera name="zed" model="zed2i" enable_gnss="false">
   <!-- block required by *gnss_origin; used only if GNSS is enabled -->
   <origin xyz="0 0 0" rpy="0 0 0"/>
 </xacro:zed_camera>
   <!-- Mount ZED to rot_link (this replaces the old 'parent' + nested origin) -->
-  <joint name="zed2i_mount" type="fixed">
+  <joint name="zed_mount" type="fixed">
     <parent link="$(arg rot_link)"/>
-    <child  link="zed2i_camera_link"/>
+    <child  link="zed_camera_link"/>
     <origin xyz="$(arg zed_xyz)" rpy="$(arg zed_rpy)"/>
   </joint>
