Commit message: addjusted lidar frame

File: urdf/ouster_os1.urdf.xacro (robot description, xacro)
@@ -41,5 +41,5 @@
       <parent link="${name}" />
       <child link="${lidar_link}" />
-      <origin xyz="0.0 0.0 0.03618" rpy="0 0 0" />
+      <origin xyz="0.0 0.0 0.03618" rpy="0 0 3.14159" />
     </joint>
     <!-- Gazebo requires the ouster_gazebo_plugins package -->
