Commit message: perfect working urdf

File: urdf/zed_macro.urdf.xacro (robot description, xacro)
@@ -191,9 +191,15 @@
       </joint>
       <!-- ZED2 Sensors -->
-      <xacro:if value="${model == 'zed2'}">
+      <xacro:if value="${model == 'zed2i'}">
         <link name="${name}_mag_link" />
         <joint name="${name}_mag_joint" type="fixed">
           <parent link="${name}_camera_center"/>
           <child link="${name}_mag_link"/>
+          <origin xyz="0 0 0" rpy="0 0 0" />
+        </joint>
+        <link name="${name}_imu_link"/>
+        <joint name="${name}_imu_joint" type="fixed">
+          <parent link="${name}_left_camera_frame"/>
+          <child  link="${name}_imu_link"/>
           <origin xyz="0 0 0" rpy="0 0 0" />
         </joint>
